Commit message: Change package name

File: dynamixel_7dof_arm_description/urdf/dynamixel_7dof_arm.gazebo.xacro (robot description, xacro)
@@ -15,6 +15,4 @@
   <!-- World -->
   <gazebo reference="world"/>
-  <!-- Link0 -->
-  <RefLink ref="link0"/>
   <!-- Link1 -->
   <RefLink ref="link1"/>

File: dynamixel_7dof_arm_description/urdf/dynamixel_7dof_arm.urdf.xacro (robot description, xacro)
@@ -2,25 +2,17 @@
 <!-- Manipulator Chain -->
 <robot xmlns:xacro="http://ros.org/wiki/xacro">
-  <!-- Link 0 -->
-  <link name="link0"/>
-  <!-- Joint 0 -->
-  <joint name="joint0" type="fixed">
-    <parent link="link0"/>
-    <child link="link1"/>
-    <origin xyz="0.0 0.0 0.0465" rpy="0 0 0"/>
-  </joint>
   <!-- Link 1 -->
   <link name="link1">
     <visual>
-      <origin xyz="0 0 0" rpy="0 0 0"/>
-      <geometry>
-        <mesh filename="package://manipulator_description/meshes/link1.stl" scale="0.001 0.001 0.001"/>
-      </geometry>
-      <material name="grey"/>
-    </visual>
-    <collision>
-      <origin xyz="0 0 0" rpy="0 0 0"/>
-      <geometry>
-        <mesh filename="package://manipulator_description/meshes/link1.stl" scale="0.001 0.001 0.001"/>
+      <origin xyz="0 0 0.044" rpy="0 0 0"/>
+      <geometry>
+        <mesh filename="package://dynamixel_7dof_arm_description/meshes/link1_visual.stl" scale="0.001 0.001 0.001"/>
+      </geometry>
+      <material name="grey"/>
+    </visual>
+    <collision>
+      <origin xyz="0 0 0.044" rpy="0 0 0"/>
+      <geometry>
+        <mesh filename="package://dynamixel_7dof_arm_description/meshes/link1_collision.stl" scale="0.001 0.001 0.001"/>
       </geometry>
     </collision>
@@ -37,5 +29,5 @@
     <parent link="link1"/>
     <child link="link2"/>
-    <origin xyz="0.012 0.0 0.017" rpy="0 0 0"/>
+    <origin xyz="0.0 0.0 0.098" rpy="-pi/2 0 0"/>
     <axis xyz="0 0 1"/>
     <limit velocity="4.8" effort="1" lower="${-pi*0.9}" upper="${pi*0.9}" />
@@ -44,14 +36,14 @@
   <link name="link2">
     <visual>
-      <origin xyz="0 0 0.019" rpy="0 0 0"/>
-      <geometry>
-        <mesh filename="package://manipulator_description/meshes/link2.stl" scale="0.001 0.001 0.001"/>
-      </geometry>
-      <material name="grey"/>
-    </visual>
-    <collision>
-      <origin xyz="0 0 0.019" rpy="0 0 0"/>
-      <geometry>
-        <mesh filename="package://manipulator_description/meshes/link2.stl" scale="0.001 0.001 0.001"/>
+      <origin xyz="0 0 0" rpy="0 0 0"/>
+      <geometry>
+        <mesh filename="package://dynamixel_7dof_arm_description/meshes/link2_visual.stl" scale="0.001 0.001 0.001"/>
+      </geometry>
+      <material name="grey"/>
+    </visual>
+    <collision>
+      <origin xyz="0 0 0" rpy="0 0 0"/>
+      <geometry>
+        <mesh filename="package://dynamixel_7dof_arm_description/meshes/link2_collision.stl" scale="0.001 0.001 0.001"/>
       </geometry>
     </collision>
@@ -68,6 +60,6 @@
     <parent link="link2"/>
     <child link="link3"/>
-    <origin xyz="0.0 0.0 0.0595" rpy="0 0 0"/>
-    <axis xyz="0 1 0"/>
+    <origin xyz="0 -0.126 0" rpy="pi/2 0 0"/>
+    <axis xyz="0 0 1"/>
     <limit velocity="4.8" effort="1" lower="${-pi*0.57}" upper="${pi*0.5}" />
   </joint>
@@ -77,12 +69,12 @@
       <origin xyz="0 0 0" rpy="0 0 0"/>
       <geometry>
-        <mesh filename="package://manipulator_description/meshes/link3.stl" scale="0.001 0.001 0.001"/>
-      </geometry>
-      <material name="grey"/>
-    </visual>
-    <collision>
-      <origin xyz="0 0 0" rpy="0 0 0"/>
-      <geometry>
-        <mesh filename="package://manipulator_description/meshes/link3.stl" scale="0.001 0.001 0.001"/>
+        <mesh filename="package://dynamixel_7dof_arm_description/meshes/link3_visual.stl" scale="0.001 0.001 0.001"/>
+      </geometry>
+      <material name="grey"/>
+    </visual>
+    <collision>
+      <origin xyz="0 0 0" rpy="0 0 0"/>
+      <geometry>
+        <mesh filename="package://dynamixel_7dof_arm_description/meshes/link3_collision.stl" scale="0.001 0.001 0.001"/>
       </geometry>
     </collision>
@@ -99,5 +91,5 @@
     <parent link="link3"/>
     <child link="link4"/>
-    <origin xyz="0.024 0 0.128" rpy="0 0 0"/>
+    <origin xyz="0 0 0.054" rpy="-pi/2 0 0"/>
     <axis xyz="0 1 0"/>
     <limit velocity="4.8" effort="1" lower="${-pi*0.3}" upper="${pi*0.44}" />
@@ -108,12 +100,12 @@
       <origin xyz="0 0 0" rpy="0 0 0"/>
       <geometry>
-        <mesh filename="package://manipulator_description/meshes/link4.stl" scale="0.001 0.001 0.001"/>
-      </geometry>
-      <material name="grey"/>
-    </visual>
-    <collision>
-      <origin xyz="0 0 0" rpy="0 0 0"/>
-      <geometry>
-        <mesh filename="package://manipulator_description/meshes/link4.stl" scale="0.001 0.001 0.001"/>
+        <mesh filename="package://dynamixel_7dof_arm_description/meshes/link4_visual.stl" scale="0.001 0.001 0.001"/>
+      </geometry>
+      <material name="grey"/>
+    </visual>
+    <collision>
+      <origin xyz="0 0 0" rpy="0 0 0"/>
+      <geometry>
+        <mesh filename="package://dynamixel_7dof_arm_description/meshes/link4_collision.stl" scale="0.001 0.001 0.001"/>
       </geometry>
     </collision>
@@ -130,5 +122,5 @@
     <parent link="link4"/>
     <child link="link5"/>
-    <origin xyz="0.124 0.0 0.0" rpy="0 0 0"/>
+    <origin xyz="0 -0.092 0" rpy="pi/2 0 0"/>
     <axis xyz="0 1 0"/>
     <limit velocity="4.8" effort="1" lower="${-pi*0.57}" upper="${pi*0.65}" />
@@ -139,12 +131,12 @@
       <origin xyz="0 0 0" rpy="0 0 0"/>
       <geometry>
-        <mesh filename="package://manipulator_description/meshes/link5.stl" scale="0.001 0.001 0.001"/>
-      </geometry>
-      <material name="grey"/>
-    </visual>
-    <collision>
-      <origin xyz="0 0 0" rpy="0 0 0"/>
-      <geometry>
-        <mesh filename="package://manipulator_description/meshes/link5.stl" scale="0.001 0.001 0.001"/>
+        <mesh filename="package://dynamixel_7dof_arm_description/meshes/link5_visual.stl" scale="0.001 0.001 0.001"/>
+      </geometry>
+      <material name="grey"/>
+    </visual>
+    <collision>
+      <origin xyz="0 0 0" rpy="0 0 0"/>
+      <geometry>
+        <mesh filename="package://dynamixel_7dof_arm_description/meshes/link5_collision.stl" scale="0.001 0.001 0.001"/>
       </geometry>
     </collision>
@@ -161,5 +153,5 @@
     <parent link="link5"/>
     <child link="link6"/>
-    <origin xyz="0.124 0.0 0.0" rpy="0 0 0"/>
+    <origin xyz="0 0 0.0425" rpy="-pi/2 0 0"/>
     <axis xyz="0 1 0"/>
     <limit velocity="4.8" effort="1" lower="${-pi*0.57}" upper="${pi*0.65}" />
@@ -170,12 +162,12 @@
       <origin xyz="0 0 0" rpy="0 0 0"/>
       <geometry>
-        <mesh filename="package://manipulator_description/meshes/link6.stl" scale="0.001 0.001 0.001"/>
-      </geometry>
-      <material name="grey"/>
-    </visual>
-    <collision>
-      <origin xyz="0 0 0" rpy="0 0 0"/>
-      <geometry>
-        <mesh filename="package://manipulator_description/meshes/link6.stl" scale="0.001 0.001 0.001"/>
+        <mesh filename="package://dynamixel_7dof_arm_description/meshes/link6_visual.stl" scale="0.001 0.001 0.001"/>
+      </geometry>
+      <material name="grey"/>
+    </visual>
+    <collision>
+      <origin xyz="0 0 0" rpy="0 0 0"/>
+      <geometry>
+        <mesh filename="package://dynamixel_7dof_arm_description/meshes/link6_collision.stl" scale="0.001 0.001 0.001"/>
       </geometry>
     </collision>
@@ -192,5 +184,5 @@
     <parent link="link6"/>
     <child link="link7"/>
-    <origin xyz="0.124 0.0 0.0" rpy="0 0 0"/>
+    <origin xyz="0 -0.062 0" rpy="pi/2 0 0"/>
     <axis xyz="0 1 0"/>
     <limit velocity="4.8" effort="1" lower="${-pi*0.57}" upper="${pi*0.65}" />
@@ -201,12 +193,12 @@
       <origin xyz="0 0 0" rpy="0 0 0"/>
       <geometry>
-        <mesh filename="package://manipulator_description/meshes/link7.stl" scale="0.001 0.001 0.001"/>
-      </geometry>
-      <material name="grey"/>
-    </visual>
-    <collision>
-      <origin xyz="0 0 0" rpy="0 0 0"/>
-      <geometry>
-        <mesh filename="package://manipulator_description/meshes/link7.stl" scale="0.001 0.001 0.001"/>
+        <mesh filename="package://dynamixel_7dof_arm_description/meshes/link7_visual.stl" scale="0.001 0.001 0.001"/>
+      </geometry>
+      <material name="grey"/>
+    </visual>
+    <collision>
+      <origin xyz="0 0 0" rpy="0 0 0"/>
+      <geometry>
+        <mesh filename="package://dynamixel_7dof_arm_description/meshes/link7_collision.stl" scale="0.001 0.001 0.001"/>
       </geometry>
     </collision>
@@ -223,5 +215,5 @@
     <parent link="link7"/>
     <child link="gripper"/>
-    <origin xyz="0.124 0.0 0.0" rpy="0 0 0"/>
+    <origin xyz="0 0 0.036" rpy="-pi/2 0 0"/>
     <axis xyz="0 1 0"/>
     <limit velocity="4.8" effort="1" lower="${-pi*0.57}" upper="${pi*0.65}" />
@@ -232,12 +224,12 @@
       <origin xyz="0 0 0" rpy="0 0 0"/>
       <geometry>
-        <mesh filename="package://manipulator_description/meshes/gripper.stl" scale="0.001 0.001 0.001"/>
-      </geometry>
-      <material name="grey"/>
-    </visual>
-    <collision>
-      <origin xyz="0 0 0" rpy="0 0 0"/>
-      <geometry>
-        <mesh filename="package://manipulator_description/meshes/gripper.stl" scale="0.001 0.001 0.001"/>
+        <mesh filename="package://dynamixel_7dof_arm_description/meshes/gripper_visual.stl" scale="0.001 0.001 0.001"/>
+      </geometry>
+      <material name="grey"/>
+    </visual>
+    <collision>
+      <origin xyz="0 0 0" rpy="0 0 0"/>
+      <geometry>
+        <mesh filename="package://dynamixel_7dof_arm_description/meshes/gripper_collision.stl" scale="0.001 0.001 0.001"/>
       </geometry>
     </collision>
@@ -254,7 +246,7 @@
     <parent link="gripper"/>
     <child link="finger_left"/>
-    <origin xyz="0.0817 0.021 0.0" rpy="0 0 0"/>
-    <axis xyz="0 1 0"/>
-    <limit velocity="4.8" effort="1" lower="-0.010" upper="0.019" />
+    <origin xyz="0 0 0.016" rpy="pi pi 0"/>
+    <axis xyz="0 0 -1"/>
+    <limit velocity="4.8" effort="1" lower="-0.016" upper="0.016" />
   </joint>
   <!-- Left finger link -->
@@ -263,5 +255,5 @@
       <origin xyz="0.0 0.0 0" rpy="0 0 0"/>
       <geometry>
-        <mesh filename="package://manipulator_description/meshes/finger.stl" scale="0.001 0.001 0.001"/>
+        <mesh filename="package://dynamixel_7dof_arm_description/meshes/finger_visual.stl" scale="0.001 0.001 0.001"/>
       </geometry>
       <material name="grey"/>
@@ -270,5 +262,5 @@
       <origin xyz="0.0 0.0 0" rpy="0 0 0"/>
       <geometry>
-        <mesh filename="package://manipulator_description/meshes/finger.stl" scale="0.001 0.001 0.001"/>
+        <mesh filename="package://dynamixel_7dof_arm_description/meshes/finger_collision.stl" scale="0.001 0.001 0.001"/>
       </geometry>
     </collision>
@@ -285,7 +277,7 @@
     <parent link="gripper"/>
     <child link="finger_right"/>
-    <origin xyz="0.0817 -0.021 0" rpy="0 0 0"/>
-    <axis xyz="0 -1 0"/>
-    <limit velocity="4.8" effort="1" lower="-0.010" upper="0.019" />
+    <origin xyz="0 0 -0.016" rpy="0 0 pi"/>
+    <axis xyz="0 0 1"/>
+    <limit velocity="4.8" effort="1" lower="-0.016" upper="0.016" />
     <mimic joint="gripper" multiplier="1"/>
   </joint>
@@ -293,14 +285,14 @@
   <link name="finger_right">
     <visual>
-      <origin xyz="0.0 -0.0 0" rpy="0 0 0"/>
-      <geometry>
-        <mesh filename="package://manipulator_description/meshes/finger.stl" scale="0.001 0.001 0.001"/>
-      </geometry>
-      <material name="grey"/>
-    </visual>
-    <collision>
-      <origin xyz="0.0 -0.0 0" rpy="0 0 0"/>
-      <geometry>
-        <mesh filename="package://manipulator_description/meshes/finger.stl" scale="0.001 0.001 0.001"/>
+      <origin xyz="0 0 0" rpy="0 0 0"/>
+      <geometry>
+        <mesh filename="package://dynamixel_7dof_arm_description/meshes/finger_visual.stl" scale="0.001 0.001 0.001"/>
+      </geometry>
+      <material name="grey"/>
+    </visual>
+    <collision>
+      <origin xyz="0 0 0" rpy="0 0 0"/>
+      <geometry>
+        <mesh filename="package://dynamixel_7dof_arm_description/meshes/finger_collision.stl" scale="0.001 0.001 0.001"/>
       </geometry>
     </collision>
@@ -315,5 +307,5 @@
   <!-- end effector joint -->
   <joint name="end_effector_joint" type="fixed">
-    <origin xyz="0.126 0.0 0.0" rpy="0 0 0"/>
+    <origin xyz="0 -0.0565 0" rpy="pi/2 0 0"/>
     <parent link="gripper"/>
     <child link="end_effector_link"/>
