Commit message: Update urdf

File: dynamixel_7dof_arm_description/urdf/dynamixel_7dof_arm.urdf.xacro (robot description, xacro)
@@ -18,9 +18,9 @@
     </collision>
     <inertial>
-      <origin xyz="3.0876154e-04 0.0000000e+00 -1.2176461e-04" />
-      <mass value="7.9119962e-02" />
-      <inertia ixx="1.2505234e-05" ixy="0.0" ixz="-1.7855208e-07"
-               iyy="2.1898364e-05" iyz="0.0"
-               izz="1.9267361e-05" />
+      <origin xyz="0 0 0.044" />
+      <mass value="1.65e-01" />
+      <inertia ixx="9.7675421e-05" ixy="1.5076192e-06" ixz="-7.0306018e-05"
+               iyy="1.9686152e-04" iyz="1.4556164e-06"
+               izz="1.2605450e-04" />
     </inertial>
   </link>
@@ -29,7 +29,7 @@
     <parent link="link1"/>
     <child link="link2"/>
-    <origin xyz="0.0 0.0 0.098" rpy="-pi/2 0 0"/>
+    <origin xyz="0.0 0.0 0.098" rpy="${-pi*0.5} 0 0"/>
     <axis xyz="0 0 1"/>
-    <limit velocity="4.8" effort="1" lower="${-pi*0.9}" upper="${pi*0.9}" />
+    <limit velocity="${pi}" effort="1" lower="${-pi*0.9}" upper="${pi*0.9}" />
   </joint>
   <!--  Link 2 -->
@@ -49,9 +49,9 @@
     </collision>
     <inertial>
-      <origin xyz="-3.0184870e-04 5.4043684e-04 ${0.018 + 2.9433464e-02}" />
-      <mass value="9.8406837e-02" />
-      <inertia ixx="3.4543422e-05" ixy="-1.6031095e-08" ixz="-3.8375155e-07"
-               iyy="3.2689329e-05" iyz="2.8511935e-08"
-               izz="1.8850320e-05" />
+      <origin xyz="0 0 0" />
+      <mass value="3.65360184e-01" />
+      <inertia ixx="7.23925638e-04" ixy="-2.9538917e-06" ixz="4.0975813308e-06"
+               iyy="4.921326352e-04" iyz="1.767767725e-04"
+               izz="3.02730708e-04" />
     </inertial>
   </link>
@@ -60,7 +60,7 @@
     <parent link="link2"/>
     <child link="link3"/>
-    <origin xyz="0 -0.126 0" rpy="pi/2 0 0"/>
+    <origin xyz="0 -0.126 0" rpy="${pi*0.5} 0 0"/>
     <axis xyz="0 0 1"/>
-    <limit velocity="4.8" effort="1" lower="${-pi*0.57}" upper="${pi*0.5}" />
+    <limit velocity="${pi}" effort="1" lower="${-pi*0.25}" upper="${pi*0.5}" />
   </joint>
   <!--  Link 3 -->
@@ -80,9 +80,9 @@
     </collision>
     <inertial>
-      <origin xyz="1.0308393e-02 3.7743363e-04 1.0170197e-01" />
-      <mass value="1.3850917e-01" />
-      <inertia ixx="3.3055381e-04" ixy="-9.7940978e-08" ixz="-3.8505711e-05"
-               iyy="3.4290447e-04" iyz="-1.5717516e-06"
-               izz="6.0346498e-05" />
+      <origin xyz="0 0 0" />
+      <mass value="2.12396196e-01" />
+      <inertia ixx="4.36697977e-04" ixy="1.5076192e-06" ixz="-8.98306422e-05"
+               iyy="5.31846236e-04" iyz="1.4556164e-06"
+               izz="1.5563934e-04" />
     </inertial>
   </link>
@@ -91,5 +91,5 @@
     <parent link="link3"/>
     <child link="link4"/>
-    <origin xyz="0 0 0.054" rpy="-pi/2 0 0"/>
+    <origin xyz="0 0 0.054" rpy="${-pi*0.5} 0 0"/>
     <axis xyz="0 1 0"/>
     <limit velocity="4.8" effort="1" lower="${-pi*0.3}" upper="${pi*0.44}" />
@@ -111,9 +111,9 @@
     </collision>
     <inertial>
-      <origin xyz="9.0909590e-02 3.8929816e-04 2.2413279e-04" />
-      <mass value="1.3274562e-01" />
-      <inertia ixx="3.0654178e-05" ixy="-1.2764155e-06" ixz="-2.6874417e-07"
-               iyy="2.4230292e-04" iyz="1.1559550e-08"
-               izz="2.5155057e-04" />
+      <origin xyz="0 0 0" />
+      <mass value="1.76006714e-01" />
+      <inertia ixx="1.69380031e-04" ixy="-1.5076192e-06" ixz="-9.8692692e-09"
+               iyy="4.53380742e-05" iyz="-1.8439349e-06"
+               izz="1.52969543e-04" />
     </inertial>
   </link>
@@ -122,5 +122,5 @@
     <parent link="link4"/>
     <child link="link5"/>
-    <origin xyz="0 -0.092 0" rpy="pi/2 0 0"/>
+    <origin xyz="0 -0.092 0" rpy="${pi*0.5} 0 0"/>
     <axis xyz="0 1 0"/>
     <limit velocity="4.8" effort="1" lower="${-pi*0.57}" upper="${pi*0.65}" />
@@ -142,9 +142,9 @@
     </collision>
     <inertial>
-      <origin xyz="9.0909590e-02 3.8929816e-04 2.2413279e-04" />
-      <mass value="1.3274562e-01" />
-      <inertia ixx="3.0654178e-05" ixy="-1.2764155e-06" ixz="-2.6874417e-07"
-               iyy="2.4230292e-04" iyz="1.1559550e-08"
-               izz="2.5155057e-04" />
+      <origin xyz="0 0 0" />
+      <mass value="1.140236536e-01" />
+      <inertia ixx="1.73149898e-04" ixy="6.4100516e-07" ixz="-5.44674084e-05"
+               iyy="2.05741025e-04" iyz="5.6194478e-07"
+               izz="6.4729774e-05" />
     </inertial>
   </link>
@@ -153,5 +153,5 @@
     <parent link="link5"/>
     <child link="link6"/>
-    <origin xyz="0 0 0.0425" rpy="-pi/2 0 0"/>
+    <origin xyz="0 0 0.0425" rpy="${-pi*0.5} 0 0"/>
     <axis xyz="0 1 0"/>
     <limit velocity="4.8" effort="1" lower="${-pi*0.57}" upper="${pi*0.65}" />
@@ -173,9 +173,9 @@
     </collision>
     <inertial>
-      <origin xyz="9.0909590e-02 3.8929816e-04 2.2413279e-04" />
-      <mass value="1.3274562e-01" />
-      <inertia ixx="3.0654178e-05" ixy="-1.2764155e-06" ixz="-2.6874417e-07"
-               iyy="2.4230292e-04" iyz="1.1559550e-08"
-               izz="2.5155057e-04" />
+      <origin xyz="0 0 0" />
+      <mass value="8.76309701e-02" />
+      <inertia ixx="5.25353043e-05" ixy="-6.4100516e-07" ixz="-5.5567317e-09"
+               iyy="1.49092849e-05" iyz="-1.0653297e-06"
+               izz="4.86901315e-05" />
     </inertial>
   </link>
@@ -184,5 +184,5 @@
     <parent link="link6"/>
     <child link="link7"/>
-    <origin xyz="0 -0.062 0" rpy="pi/2 0 0"/>
+    <origin xyz="0 -0.062 0" rpy="${pi*0.5} 0 0"/>
     <axis xyz="0 1 0"/>
     <limit velocity="4.8" effort="1" lower="${-pi*0.57}" upper="${pi*0.65}" />
@@ -204,9 +204,9 @@
     </collision>
     <inertial>
-      <origin xyz="9.0909590e-02 3.8929816e-04 2.2413279e-04" />
-      <mass value="1.3274562e-01" />
-      <inertia ixx="3.0654178e-05" ixy="-1.2764155e-06" ixz="-2.6874417e-07"
-               iyy="2.4230292e-04" iyz="1.1559550e-08"
-               izz="2.5155057e-04" />
+      <origin xyz="0 0 0" />
+      <mass value="9.3693466e-02" />
+      <inertia ixx="5.2902474e-05" ixy="6.40951087082e-07" ixz="-2.4025384e-05"
+               iyy="8.2881293e-05" iyz="5.6194478e-07"
+               izz="4.61038615e-05" />
     </inertial>
   </link>
@@ -215,5 +215,5 @@
     <parent link="link7"/>
     <child link="gripper"/>
-    <origin xyz="0 0 0.036" rpy="-pi/2 0 0"/>
+    <origin xyz="0 0 0.036" rpy="${-pi*0.5} 0 0"/>
     <axis xyz="0 1 0"/>
     <limit velocity="4.8" effort="1" lower="${-pi*0.57}" upper="${pi*0.65}" />
@@ -235,9 +235,9 @@
     </collision>
     <inertial>
-      <origin xyz="4.4206755e-02 3.6839985e-07 8.9142216e-03" />
-      <mass value="1.4327573e-01" />
-      <inertia ixx="8.0870749e-05" ixy="0.0" ixz="-1.0157896e-06"
-               iyy="7.5980465e-05" iyz="0.0"
-               izz="9.3127351e-05" />
+      <origin xyz="0 0 0" />
+      <mass value="1.175366352e-01" />
+      <inertia ixx="6.087557e-05" ixy="-5.0302e-08" ixz="-2.027965366431884e-05"
+               iyy="9.5134911e-05" iyz="5.61960245365e-07"
+               izz="4.986382864e-05" />
     </inertial>
   </link>
@@ -246,5 +246,5 @@
     <parent link="gripper"/>
     <child link="finger_left"/>
-    <origin xyz="0 0 0.016" rpy="pi pi 0"/>
+    <origin xyz="0 0 0.016" rpy="${pi} ${pi} 0"/>
     <axis xyz="0 0 -1"/>
     <limit velocity="4.8" effort="1" lower="-0.016" upper="0.016" />
@@ -253,5 +253,5 @@
   <link name="finger_left">
     <visual>
-      <origin xyz="0.0 0.0 0" rpy="0 0 0"/>
+      <origin xyz="0 0 0" rpy="0 0 0"/>
       <geometry>
         <mesh filename="package://dynamixel_7dof_arm_description/meshes/finger_visual.stl" scale="0.001 0.001 0.001"/>
@@ -260,5 +260,5 @@
     </visual>
     <collision>
-      <origin xyz="0.0 0.0 0" rpy="0 0 0"/>
+      <origin xyz="0 0 0" rpy="0 0 0"/>
       <geometry>
         <mesh filename="package://dynamixel_7dof_arm_description/meshes/finger_collision.stl" scale="0.001 0.001 0.001"/>
@@ -267,8 +267,8 @@
     <inertial>
       <origin xyz="0 0 0" />
-      <mass value="1.0e-03" />
-      <inertia ixx="1.0e-03" ixy="0.0" ixz="0.0"
-               iyy="1.0e-03" iyz="0.0"
-               izz="1.0e-03" />
+      <mass value="1.5157383e-02" />
+      <inertia ixx="2.1703323e-06" ixy="4.7785008e-08" ixz="1.9357889e-06"
+               iyy="1.4304498e-05" iyz="1.8450264e-07"
+               izz="1.3405196e-05" />
     </inertial>
   </link>
@@ -277,5 +277,5 @@
     <parent link="gripper"/>
     <child link="finger_right"/>
-    <origin xyz="0 0 -0.016" rpy="0 0 pi"/>
+    <origin xyz="0 0 -0.016" rpy="0 0 ${pi}"/>
     <axis xyz="0 0 1"/>
     <limit velocity="4.8" effort="1" lower="-0.016" upper="0.016" />
@@ -299,13 +299,13 @@
     <inertial>
       <origin xyz="0 0 0" />
-      <mass value="1.0e-03" />
-      <inertia ixx="1.0e-03" ixy="0.0" ixz="0.0"
-               iyy="1.0e-03" iyz="0.0"
-               izz="1.0e-03" />
+      <mass value="1.5157383e-02" />
+      <inertia ixx="2.1703323e-06" ixy="4.7785008e-08" ixz="1.9357889e-06"
+               iyy="1.4304498e-05" iyz="1.8450264e-07"
+               izz="1.3405196e-05" />
     </inertial>
   </link>
   <!-- end effector joint -->
   <joint name="end_effector_joint" type="fixed">
-    <origin xyz="0 -0.0565 0" rpy="pi/2 0 0"/>
+    <origin xyz="0 -0.0565 0" rpy="${pi/2} 0 0"/>
     <parent link="gripper"/>
     <child link="end_effector_link"/>
